Commit message: cartpole1

File: urdf/cartpole.xacro (robot description, xacro)
@@ -2,4 +2,13 @@
 <robot name="cartpole" xmlns:xacro="http://www.ros.org/wiki/xacro">
 	<static>true</static>
+<link name="world"/>
+<joint name=" chassis_world" type="prismatic">
+    <origin xyz="0 0 1" rpy="0 0 0"></origin>
+    <parent link="world"></parent>
+    <child link="link_chassis"></child>
+    <axis xyz="1 0 0"></axis>
+    <limit effort="300" lower="-500.0" upper="500.0" velocity="7.0"></limit>
+    <dynamics damping="0.0" friction="0.1"/>
+</joint>
 	<link name="link_chassis">
     <!-- pose and inertial -->
@@ -23,9 +32,10 @@
 	    </visual>
     </link>
-  <joint name="joint" type="continuous">
+  <joint name="pole_chassis" type="continuous">
       <axis xyz="0 1 0" rpy="0 0 0" />
       <parent link="link_chassis"/>
       <child link="pole"/>
       <origin xyz="0 0 0" rpy="0 0 0"/>
+	  <dynamics damping="0.0" friction="0.01"/>
   </joint>
   <link name="pole">
@@ -35,5 +45,5 @@
 	      <inertia ixx="0.02086667" ixy="0" ixz="0" iyy="0.02086667" iyz="0" izz="6.6667e-4"/>
 	    </inertial>
-	    <collision >
+	   <collision >
 	    <origin rpy="0 0 0" xyz="0 0 0.25"/>
 	      <geometry>
@@ -49,8 +59,24 @@
 	    </visual>
     </link>
-    <plugin name="joint_state_publisher" filename="libgazebo_ros_joint_state_publisher.so">
-   <jointName>joint</jointName>
+<plugin name="joint_state_publisher" filename="libgazebo_ros_joint_state_publisher.so">
+   <jointName>pole_chassis</jointName>
    <updateRate>50.0	</updateRate>
    <alwaysOn>true</alwaysOn>
 </plugin>
+  <gazebo reference="link_chassis">
+     <material>Gazebo/Red</material>
+  </gazebo>
+    <gazebo reference="pole">
+       <material>Gazebo/Orange</material>
+    </gazebo>
+<transmission name="tran1">
+    <type>transmission_interface/SimpleTransmission</type>
+    <joint name="chassis_world">
+      <hardwareInterface>EffortJointInterface</hardwareInterface>
+    </joint>
+    <actuator name="motor1">
+      <hardwareInterface>EffortJointInterface</hardwareInterface>
+      <mechanicalReduction>1</mechanicalReduction>
+    </actuator>
+  </transmission>
 </robot>

File: urdf/wall.xacro (robot description, xacro)
@@ -28,5 +28,5 @@
 	    </visual>
     </link>
-    <joint name="fixed2" type="fixed">
+  <joint name="fixed2" type="fixed">
     <parent link="world"/>
     <child link="wall2"/>
